File: public/csa/vdc/csa_vdc_v1.4d.brd (EAGLE design)
At the start: 160 x 100 mm, 59 parts, among them IC1 74HC374N, IC10 74HCT166N, IC11 74LS273BUSOPT, IC12 74HCT175N, IC13 74LS86N, IC14 74HCT74N, IC15 74HCT04N, IC16 74HCT00N, IC17 74LS32N, IC2 74HCT138N, IC21 74HCT04N, IC22 CRTC6545SMALLPADS, IC23 74HCT00N, IC24 27C128P, IC3 74LS688BUSOPT, IC4 74HCT257N, IC5 74HCT257N, IC6 74HCT257N, IC7 74HCT257N, IC8 74HCT257N, IC9 74HCT245N

Commit message: finalize vdc 1.4d
Connections:
- net N$24 renamed REGCLK
- net N$46 renamed CA13
- removed net N$23: IC12.9, IC14.9, IC23.1
- removed net N$49: IC11.2, JP10.3
- new net DECLK: IC12.9, IC14.8
- new net N$47: IC14.9, IC23.1
- net GND: now also JP10.3
Routing:
- net N$49: track 102.3 -> 0.00 mm, vias 4 -> 0
- net N$23: track 87.5 -> 0.00 mm, vias 1 -> 0
- net N$47: track 0.00 -> 72.9 mm, vias 0 -> 1
- net DECLK: track 0.00 -> 14.4 mm
- net GND: track 1219.5 -> 1233.5 mm, vias 22 -> 24
- net BD0: track 340.1 -> 341.6 mm
- net BD7: track 236.3 -> 236.9 mm
