File: public/csa/vdc/csa_vdc_v1.4d.sch (EAGLE design)
At the start: 59 parts, among them IC1 74HC374N, IC10 74HCT166N, IC11 74LS273BUSOPT, IC12 74HCT175N, IC13 74LS86N, IC14 74HCT74N, IC15 74HCT04N, IC16 74HCT00N, IC17 74LS32N, IC2 74HCT138N, IC21 74HCT04N, IC22 CRTC6545SMALLPADS, IC23 74HCT00N, IC24 27C128P, IC3 74LS688BUSOPT, IC4 74HCT257N, IC5 74HCT257N, IC6 74HCT257N, IC7 74HCT257N, IC8 74HCT257N, IC9 74HCT245N

Commit message: finalize vdc 1.4d
Connections:
- net N$24 renamed REGCLK
- net N$46 renamed CA13
- removed net N$23: IC12A.CLK, IC14B.Q, IC23A.I0
- removed net N$49: IC11G$1.Q1, JP10.3
- new net DECLK: IC12A.CLK, IC14B.!Q
- new net N$47: IC14B.Q, IC23A.I0
- net GND: now also JP10.3
Other:
- note added: "1.4D: use IC14B./Q for delaying DE/CE"
- note added: "CSA-VDC40/80-V1.4D-20211018"
- note added: "Make JP10 more reasonable, freeing ctrl port bit 7"
- note removed: "1.4D: use IC14B.Q for delaying DE/CE"
- note removed: "CSA-VDC40/80-V1.4D-20210403"
